File: projection_src_v1/dlp_projection_board_v1/dlp_displayboard.kicad_sch (KiCad schematic)
At the start: 2 parts, among them U1 DLPC3433CZVB, U2 DLPA3000DPFD

Commit message: Added 471TP and 6540 symbols
Parts:
- removed U1: DLPC3433CZVB, ZVB176_TEX, symbol DLPC3433:DLPC3433CZVB
- removed U2: DLPA3000DPFD, PFD100_TEX, symbol DLPA3000:DLPA3000DPFD

Commit message: Added DMD, Controller and Driver symbols
Parts:
- added U2: DLPC6540ZDC, BGA_40ZDC_TEX, symbol DLP6540:DLPC6540ZDC
- added U4: DLPA3005DPFD, PFD100_TEX, symbol DLPA3005:DLPA3005DPFD
